File: pcb/ReachBetween.kicad_pcb (KiCad board)
At the start: 2 copper layers, 51.8 x 73.5 mm, 11 parts, among them J1 IN, J2 Out A, J3 Out B

Commit message: Update version number correspondingly on source PCB
Other:
- board text added: "RB02 v1.1.2 © Will Harris-Braun 2022-04-17"
- board text removed: "RB02 v1.1.0 © Will Harris-Braun 2022-04-17"
Changed lines of the file:
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@@
     (effects (font (size 1.5 1.3) (thickness 0.3)) (justify mirror))
   )
-  (gr_text "RB02 v1.1.0\n© Will Harris-Braun\n2022-04-17" (at 142.5 94.2) (layer "B.SilkS")
+  (gr_text "RB02 v1.1.2\n© Will Harris-Braun\n2022-04-17" (at 142.5 94.2) (layer "B.SilkS")
     (effects (font (size 1 0.8) (thickness 0.1)) (justify left mirror))
   )

Commit message: Round silkscreen lines on back
Other:
- board text added: "RB02 v1.1.3 © Will Harris-Braun 2022-04-17"
- board text removed: "RB02 v1.1.2 © Will Harris-Braun 2022-04-17"
Changed lines of the file:
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@@
     ) (layer "B.SilkS") (width 0.025) (fill solid))
   (gr_rect (start 151 117.7) (end 149 119.7) (layer "B.SilkS") (width 0) (fill solid))
-  (gr_line (start 143.75 89.7) (end 138.5 85.7) (layer "B.SilkS") (width 2))
   (gr_poly
     (pts
@@
     ) (layer "B.SilkS") (width 0.025) (fill solid))
   (gr_rect (start 149 126.2) (end 151 124.2) (layer "B.SilkS") (width 0) (fill solid))
+  (gr_line (start 143.5 89.7) (end 142.45 88.85) (layer "B.SilkS") (width 2))
   (gr_line (start 150 101.8) (end 150 118.7) (layer "B.SilkS") (width 2))
+  (gr_poly
+    (pts
+      (xy 156.598685 88.331702)
+      (xy 155.037824 89.582187)
+      (xy 156.288309 91.143048)
+      (xy 157.84917 89.892563)
+    ) (layer "B.SilkS") (width 0) (fill solid))
+  (gr_line (start 138.5 69.25) (end 138.4 80.9) (layer "B.SilkS") (width 2))
   (gr_rect (start 149 102.7) (end 151 100.7) (layer "B.SilkS") (width 0) (fill solid))
-  (gr_line (start 161.5 85.7) (end 161.5 69.25) (layer "B.SilkS") (width 2))
+  (gr_line (start 157.55 88.85) (end 156.5 89.7) (layer "B.SilkS") (width 2))
   (gr_poly
     (pts
@@
     ) (layer "B.SilkS") (width 0.025) (fill solid))
   (gr_line (start 150 125.3) (end 150 130.75) (layer "B.SilkS") (width 2))
+  (gr_arc (start 161.6 80.9) (mid 160.54215 85.367699) (end 157.55 88.85) (layer "B.SilkS") (width 2))
   (gr_poly
     (pts
@@
       (xy 139.95605 109.05397)
     ) (layer "B.SilkS") (width 0.025) (fill solid))
-  (gr_line (start 161.5 85.7) (end 156.5 89.7) (layer "B.SilkS") (width 2))
-  (gr_line (start 138.5 85.25) (end 138.5 69.25) (layer "B.SilkS") (width 2))
   (gr_poly
     (pts
@@
       (xy 140.27732 108.324382)
     ) (layer "B.SilkS") (width 0.025) (fill solid))
+  (gr_arc (start 142.45 88.85) (mid 139.457841 85.367703) (end 138.4 80.9) (layer "B.SilkS") (width 2))
   (gr_poly
     (pts
@@
       (xy 137.557997 109.051969)
     ) (layer "B.SilkS") (width 0.025) (fill solid))
+  (gr_line (start 161.6 80.9) (end 161.5 69.25) (layer "B.SilkS") (width 2))
+  (gr_poly
+    (pts
+      (xy 143.401315 88.331702)
+      (xy 144.962176 89.582187)
+      (xy 143.711691 91.143048)
+      (xy 142.15083 89.892563)
+    ) (layer "B.SilkS") (width 0) (fill solid))
   (gr_poly
     (pts
@@
       (xy 140.568361 109.05397)
     ) (layer "B.SilkS") (width 0.025) (fill solid))
-  (gr_poly
-    (pts
-      (xy 145.157798 89.511062)
-      (xy 143.566851 88.299085)
-      (xy 142.354874 89.890032)
-      (xy 143.945821 91.102009)
-    ) (layer "B.SilkS") (width 0) (fill solid))
-  (gr_poly
-    (pts
-      (xy 156.598685 88.331702)
-      (xy 155.037824 89.582187)
-      (xy 156.288309 91.143048)
-      (xy 157.84917 89.892563)
-    ) (layer "B.SilkS") (width 0) (fill solid))
   (gr_line locked (start 175.700633 111.737867) (end 157.850774 136.33265) (layer "Edge.Cuts") (width 0.2))
   (gr_line locked (start 157.041455 136.745281) (end 142.958545 136.74528) (layer "Edge.Cuts") (width 0.2))
@@
     (effects (font (size 1.5 1.3) (thickness 0.3)) (justify mirror))
   )
-  (gr_text "RB02 v1.1.2\n© Will Harris-Braun\n2022-04-17" (at 142.5 94.2) (layer "B.SilkS")
+  (gr_text "RB02 v1.1.3\n© Will Harris-Braun\n2022-04-17" (at 142.5 94.2) (layer "B.SilkS")
     (effects (font (size 1 0.8) (thickness 0.1)) (justify left mirror))
   )
